File: usbtiny.sch (KiCad schematic (older format))
At the start: 20 parts, among them IC1 ATTINY2313-P, P1 CONN_01X01, P2 USB_A, P3 CONN_01X06, Y1 12MHz

Commit message: * Added png schematic and PCB * Added Attiny hex image and flash script
Parts:
- removed P1: CONN_01X01, symbol CONN_01X01
- C1, C2, C3: footprint (none) -> Capacitors_SMD:C_1206_HandSoldering
- D1, D2: footprint (none) -> LEDs:LED_0805
- IC1: footprint DIP20 -> Housings_DIP:DIP-20_W7.62mm
- P2: footprint (none) -> Connect:USB_A
- P3: footprint (none) -> Pin_Headers:Pin_Header_Straight_1x06
- R1, R10, R2, R3, R4, R5, R6, R7, R8: footprint (none) -> Resistors_SMD:R_0805
- R9: value 1K -> 1K5; footprint (none) -> Resistors_SMD:R_0805
- Y1: footprint (none) -> Crystals:Crystal_HC49-U_Vertical
Connections:
- net at IC1.16 ((PCINT4/OC1B)PB4): now also R7.1; no longer R4.1
- net at IC1.17 ((PCINT5/MOSI/DI/SDA)PB5): now also R6.1; no longer R5.1
- net at IC1.18 ((PCINT6/MISO/DO)PB6): now also R5.1; no longer R6.1
- net at IC1.19 ((PCINT7/USCK/SCK/SCL)PB7): now also R4.1; no longer R7.1
Changed lines of the file:
@@
 LIBS:contrib
 LIBS:valves
+LIBS:usbtiny-cache
 EELAYER 25 0
 EELAYER END
@@
 F 0 "IC1" H 2650 3850 50  0000 C CNN
 F 1 "ATTINY2313-P" H 4400 1950 50  0000 C CNN
-F 2 "DIP20" H 3600 2850 50  0000 C CIN
+F 2 "Housings_DIP:DIP-20_W7.62mm" H 3600 2850 50  0000 C CIN
 F 3 "" H 3600 2850 50  0000 C CNN
 	1    3600 2850
@@
 F 0 "Y1" H 2050 2600 50  0000 C CNN
 F 1 "12MHz" H 2050 2300 50  0000 C CNN
-F 2 "" H 2050 2450 50  0000 C CNN
+F 2 "Crystals:Crystal_HC49-U_Vertical" H 2050 2450 50  0001 C CNN
 F 3 "" H 2050 2450 50  0000 C CNN
 	1    2050 2450
@@
 F 0 "C1" H 2110 2120 50  0000 L CNN
 F 1 "22p" H 2110 1970 50  0000 L CNN
-F 2 "" H 2100 2050 50  0000 C CNN
+F 2 "Capacitors_SMD:C_1206_HandSoldering" H 2100 2050 50  0001 C CNN
 F 3 "" H 2100 2050 50  0000 C CNN
 	1    2100 2050
@@
 F 0 "C2" H 2110 2870 50  0000 L CNN
 F 1 "22p" H 2110 2720 50  0000 L CNN
-F 2 "" H 2100 2800 50  0000 C CNN
+F 2 "Capacitors_SMD:C_1206_HandSoldering" H 2100 2800 50  0001 C CNN
 F 3 "" H 2100 2800 50  0000 C CNN
 	1    2100 2800
@@
 F 0 "R1" V 2530 1200 50  0000 C CNN
 F 1 "10K" V 2450 1200 50  0000 C CNN
-F 2 "" V 2380 1200 50  0000 C CNN
+F 2 "Resistors_SMD:R_0805" V 2380 1200 50  0001 C CNN
 F 3 "" H 2450 1200 50  0000 C CNN
 	1    2450 1200
@@
 F 0 "C3" H 3060 1270 50  0000 L CNN
 F 1 "100n" H 3060 1120 50  0000 L CNN
-F 2 "" H 3050 1200 50  0000 C CNN
+F 2 "Capacitors_SMD:C_1206_HandSoldering" H 3050 1200 50  0001 C CNN
 F 3 "" H 3050 1200 50  0000 C CNN
 	1    3050 1200
@@
 F 0 "P2" H 6950 2200 50  0000 C CNN
 F 1 "USB_A" H 6700 2600 50  0000 C CNN
-F 2 "" V 6700 2300 50  0000 C CNN
+F 2 "Connect:USB_A" V 6700 2300 50  0001 C CNN
 F 3 "" V 6700 2300 50  0000 C CNN
 	1    6750 2400
@@
 F 0 "R10" V 7280 2350 50  0000 C CNN
 F 1 "1K" V 7200 2350 50  0000 C CNN
-F 2 "" V 7130 2350 50  0000 C CNN
+F 2 "Resistors_SMD:R_0805" V 7130 2350 50  0001 C CNN
 F 3 "" H 7200 2350 50  0000 C CNN
 	1    7200 2350
@@
 F 0 "D2" H 7200 2950 50  0000 C CNN
 F 1 "LED" H 7200 2750 50  0000 C CNN
-F 2 "" H 7200 2850 50  0000 C CNN
+F 2 "LEDs:LED_0805" H 7200 2850 50  0001 C CNN
 F 3 "" H 7200 2850 50  0000 C CNN
 	1    7200 2850
@@
 F 0 "R2" V 5180 3450 50  0000 C CNN
 F 1 "1K" V 5100 3450 50  0000 C CNN
-F 2 "" V 5030 3450 50  0000 C CNN
+F 2 "Resistors_SMD:R_0805" V 5030 3450 50  0001 C CNN
 F 3 "" H 5100 3450 50  0000 C CNN
 	1    5100 3450
@@
 F 0 "D1" H 5750 3350 50  0000 C CNN
 F 1 "LED" H 5600 3350 50  0000 C CNN
-F 2 "" H 5600 3450 50  0000 C CNN
+F 2 "LEDs:LED_0805" H 5600 3450 50  0001 C CNN
 F 3 "" H 5600 3450 50  0000 C CNN
 	1    5600 3450
@@
 F 0 "R8" V 6200 2750 50  0000 C CNN
 F 1 "27R-47R" V 6200 3000 50  0000 C CNN
-F 2 "" V 6030 2850 50  0000 C CNN
+F 2 "Resistors_SMD:R_0805" V 6030 2850 50  0001 C CNN
 F 3 "" H 6100 2850 50  0000 C CNN
 	1    6100 2850
@@
 F 0 "R3" V 6050 2950 50  0000 C CNN
 F 1 "27-47R" V 6050 2700 50  0000 C CNN
-F 2 "" V 5880 2850 50  0000 C CNN
+F 2 "Resistors_SMD:R_0805" V 5880 2850 50  0001 C CNN
 F 3 "" H 5950 2850 50  0000 C CNN
 	1    5950 2850
@@
 P 6400 3250
 F 0 "R9" V 6480 3250 50  0000 C CNN
-F 1 "1K" V 6400 3250 50  0000 C CNN
-F 2 "" V 6330 3250 50  0000 C CNN
+F 1 "1K5" V 6400 3250 50  0000 C CNN
+F 2 "Resistors_SMD:R_0805" V 6330 3250 50  0001 C CNN
 F 3 "" H 6400 3250 50  0000 C CNN
 	1    6400 3250
@@
 F 0 "P3" H 6850 1800 50  0000 C CNN
 F 1 "CONN_01X06" V 6950 1450 50  0000 C CNN
-F 2 "" H 6850 1450 50  0000 C CNN
+F 2 "Pin_Headers:Pin_Header_Straight_1x06" H 6850 1450 50  0001 C CNN
 F 3 "" H 6850 1450 50  0000 C CNN
 	1    6850 1450
 	1    0    0    -1
 $EndComp
-Wire Wire Line
-	6450 1200 6650 1200
-Connection ~ 6450 1200
 $Comp
 L GNDREF #PWR09
 U 1 1 5809FED5
-P 6650 1800
-F 0 "#PWR09" H 6650 1550 50  0001 C CNN
-F 1 "GNDREF" H 6950 1700 50  0000 C CNN
-F 2 "" H 6650 1800 50  0000 C CNN
-F 3 "" H 6650 1800 50  0000 C CNN
-	1    6650 1800
-	1    0    0    -1
-$EndComp
-Wire Wire Line
-	6650 1800 6650 1700
-Connection ~ 2450 1650
-$Comp
-L CONN_01X01 P1
-U 1 1 580A004F
-P 2650 1650
-F 0 "P1" H 2650 1750 50  0000 C CNN
-F 1 "CONN_01X01" V 2750 1650 50  0000 C CNN
-F 2 "" H 2650 1650 50  0000 C CNN
-F 3 "" H 2650 1650 50  0000 C CNN
-	1    2650 1650
-	1    0    0    -1
+P 6650 1700
+F 0 "#PWR09" H 6650 1450 50  0001 C CNN
+F 1 "GNDREF" V 6650 1350 50  0000 C CNN
+F 2 "" H 6650 1700 50  0000 C CNN
+F 3 "" H 6650 1700 50  0000 C CNN
+	1    6650 1700
+	0    1    1    0
 $EndComp
 Wire Wire Line
 	4750 2450 4850 2450
 Wire Wire Line
-	4850 2450 4850 1300
-Wire Wire Line
 	4750 2550 4950 2550
 Wire Wire Line
-	4950 2550 4950 1400
-Wire Wire Line
-	4750 2650 5050 2650
-Wire Wire Line
-	5050 2650 5050 1500
+	5050 2650 4750 2650
+Wire Wire Line
+	5050 1400 5050 2650
 Wire Wire Line
 	4750 2750 5150 2750
-Wire Wire Line
-	5150 2750 5150 1600
 $Comp
 L R R4
@@
 F 0 "R4" V 6100 1100 50  0000 C CNN
 F 1 "100R" V 6050 1300 50  0000 C CNN
-F 2 "" V 5980 1300 50  0000 C CNN
+F 2 "Resistors_SMD:R_0805" V 5980 1300 50  0001 C CNN
 F 3 "" H 6050 1300 50  0000 C CNN
 	1    6050 1300
@@
 F 0 "R5" V 6100 1200 50  0000 C CNN
 F 1 "100R" V 6050 1400 50  0000 C CNN
-F 2 "" V 5980 1400 50  0000 C CNN
+F 2 "Resistors_SMD:R_0805" V 5980 1400 50  0001 C CNN
 F 3 "" H 6050 1400 50  0000 C CNN
 	1    6050 1400
@@
 F 0 "R6" V 6100 1300 50  0000 C CNN
 F 1 "100R" V 6050 1500 50  0000 C CNN
-F 2 "" V 5980 1500 50  0000 C CNN
+F 2 "Resistors_SMD:R_0805" V 5980 1500 50  0001 C CNN
 F 3 "" H 6050 1500 50  0000 C CNN
 	1    6050 1500
@@
 F 0 "R7" V 6100 1400 50  0000 C CNN
 F 1 "100R" V 6050 1600 50  0000 C CNN
-F 2 "" V 5980 1600 50  0000 C CNN
+F 2 "Resistors_SMD:R_0805" V 5980 1600 50  0001 C CNN
 F 3 "" H 6050 1600 50  0000 C CNN
 	1    6050 1600
@@
 	6200 1600 6650 1600
 Wire Wire Line
-	5150 1600 5900 1600
-Wire Wire Line
-	5050 1500 5900 1500
-Wire Wire Line
-	4950 1400 5900 1400
-Wire Wire Line
-	4850 1300 5900 1300
+	4850 1600 5900 1600
+$Comp
+L PWR_FLAG #FLG010
+U 1 1 580A0BFF
+P 2700 1000
+F 0 "#FLG010" H 2700 1095 50  0001 C CNN
+F 1 "PWR_FLAG" H 2700 1180 50  0000 C CNN
+F 2 "" H 2700 1000 50  0000 C CNN
+F 3 "" H 2700 1000 50  0000 C CNN
+	1    2700 1000
+	1    0    0    -1
+$EndComp
+Connection ~ 2700 1000
+Wire Wire Line
+	5150 2750 5150 1300
+Wire Wire Line
+	4850 2450 4850 1600
+Wire Wire Line
+	5050 1400 5900 1400
+Wire Wire Line
+	4950 1500 5900 1500
+Wire Wire Line
+	4950 2550 4950 1500
+Wire Wire Line
+	5150 1300 5900 1300
+Wire Wire Line
+	6650 1200 6450 1200
+Connection ~ 6450 1200
 $EndSCHEMATC
